File: Front/MIDI_USB_Front.sch (KiCad schematic (older format))
At the start: 7 parts, among them J1 Jack_3.5mm, J2 Jack_3.5mm, J3 Jack_3.5mm, J4 Jack_3.5mm

Commit message: Add custom footprints
Parts:
- H1: footprint CustomLib:USB_C_Hole -> Custom_FP:USB_C_Hole
- H2, H3: footprint CustomLib:Wide_M3 -> Custom_FP:Wide_M3
Changed lines of the file:
@@
 F 0 "H2" H 3950 1496 50  0000 L CNN
 F 1 "MountingHole" H 3950 1405 50  0000 L CNN
-F 2 "CustomLib:Wide_M3" H 3850 1450 50  0001 C CNN
+F 2 "Custom_FP:Wide_M3" H 3850 1450 50  0001 C CNN
 F 3 "~" H 3850 1450 50  0001 C CNN
 	1    3850 1450
@@
 F 0 "H3" H 3950 1796 50  0000 L CNN
 F 1 "MountingHole" H 3950 1705 50  0000 L CNN
-F 2 "CustomLib:Wide_M3" H 3850 1750 50  0001 C CNN
+F 2 "Custom_FP:Wide_M3" H 3850 1750 50  0001 C CNN
 F 3 "~" H 3850 1750 50  0001 C CNN
 	1    3850 1750
@@
 F 0 "H1" H 3000 1946 50  0000 L CNN
 F 1 "USB hole" H 3000 1855 50  0000 L CNN
-F 2 "CustomLib:USB_C_Hole" H 2900 1900 50  0001 C CNN
+F 2 "Custom_FP:USB_C_Hole" H 2900 1900 50  0001 C CNN
 F 3 "~" H 2900 1900 50  0001 C CNN
 	1    2900 1900
