File: Front/MIDI_USB_Front.kicad_sch (KiCad schematic)
At the start: 7 parts, among them J1 Jack_3.5mm, J2 Jack_3.5mm, J3 Jack_3.5mm, J4 Jack_3.5mm

Commit message: Update front panel layout
Parts:
- added H4: Tactile hole, Custom_FP:TactileHole, symbol Mechanical:MountingHole
Changed lines of the file:
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@@
+    )
+  )
+  (symbol (lib_id "Mechanical:MountingHole") (at 73.66 59.69 0) (unit 1)
+    (in_bom yes) (on_board yes) (dnp no)
+    (property "Reference" "H4" (at 76.2 58.5216 0)
+      (effects (font (size 1.27 1.27)) (justify left))
+    )
+    (property "Value" "Tactile hole" (at 76.2 60.833 0)
+      (effects (font (size 1.27 1.27)) (justify left))
+    )
+    (property "Footprint" "Custom_FP:TactileHole" (at 73.66 59.69 0)
+      (effects (font (size 1.27 1.27)) hide)
+    )
+    (property "Datasheet" "~" (at 73.66 59.69 0)
+      (effects (font (size 1.27 1.27)) hide)
+    )
+    (instances
+      (project "MIDI_USB_Front"
+        (path "/348a85f4-2614-491e-8b4b-55e283f94479"
+          (reference "H4") (unit 1)
+        )
+      )
     )
   )

Commit message: Update metadata
Other:
- company: (none) -> GuavTek
- title: (none) -> M2IDI - USB FRONT
Changed lines of the file:
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@@
 (kicad_sch (version 20230121) (generator eeschema)
   (paper "A4")
+  (title_block
+    (title "M2IDI - USB FRONT")
+    (date "2023-06-18")
+    (rev "2.0")
+    (company "GuavTek")
+  )
   (junction (at 119.38 50.8) (diameter 0) (color 0 0 0 0)
   )
