File: Core/USB.sch (KiCad schematic (older format))
At the start: 20 parts, among them J5 USB_C_Receptacle_USB2.0, Q3 SQ2361, Q4 2N7002, U2 MIC2005-2YM5, U3 TUSB320

Commit message: Fix symbols
Parts:
- U2: symbol Custom:MIC2005 -> CustomLib:MIC2005
Changed lines of the file:
@@
 	6650 2100 6700 2100
 $Comp
-L Custom:MIC2005 U2
+L CustomLib:MIC2005 U2
 U 1 1 6099B017
 P 2900 4450

Commit message: Include symbol library
Parts:
- U2: symbol CustomLib:MIC2005 -> Custom_Sym:MIC2005
Changed lines of the file:
@@
 	6650 2100 6700 2100
 $Comp
-L CustomLib:MIC2005 U2
+L Custom_Sym:MIC2005 U2
 U 1 1 6099B017
 P 2900 4450

Commit message: Add custom footprints
Parts:
- J5: footprint CustomLib:USB_C_Receptacle_GCT_USB4085_Slimmed -> Custom_FP:USB_C_Receptacle_GCT_USB4085_Slimmed
Changed lines of the file:
@@
 F 0 "J5" H 6870 2639 50  0000 R CNN
 F 1 "USB_C_Receptacle_USB2.0" H 6870 2548 50  0000 R CNN
-F 2 "CustomLib:USB_C_Receptacle_GCT_USB4085_Slimmed" H 7450 2700 50  0001 C CNN
+F 2 "Custom_FP:USB_C_Receptacle_GCT_USB4085_Slimmed" H 7450 2700 50  0001 C CNN
 F 3 "https://www.usb.org/sites/default/files/documents/usb_type-c.zip" H 7450 2700 50  0001 C CNN
 	1    7300 2700

Commit message: Change to SMD USB connector
Parts:
- J5: footprint Custom_FP:USB_C_Receptacle_GCT_USB4085_Slimmed -> Connector_USB:USB_C_Receptacle_XKB_U262-16XN-4BVC11
Changed lines of the file:
@@
 F 0 "J5" H 6870 2639 50  0000 R CNN
 F 1 "USB_C_Receptacle_USB2.0" H 6870 2548 50  0000 R CNN
-F 2 "Custom_FP:USB_C_Receptacle_GCT_USB4085_Slimmed" H 7450 2700 50  0001 C CNN
+F 2 "Connector_USB:USB_C_Receptacle_XKB_U262-16XN-4BVC11" H 7450 2700 50  0001 C CNN
 F 3 "https://www.usb.org/sites/default/files/documents/usb_type-c.zip" H 7450 2700 50  0001 C CNN
 	1    7300 2700

Commit message: Update to v1.1
Parts:
- J5: footprint Connector_USB:USB_C_Receptacle_XKB_U262-16XN-4BVC11 -> Connector_USB:USB_C_Receptacle_HRO_TYPE-C-31-M-12
Changed lines of the file:
@@
 $Descr A4 11693 8268
 encoding utf-8
-Sheet 2 4
+Sheet 1 1
 Title ""
 Date ""
@@
 F 0 "J5" H 6870 2639 50  0000 R CNN
 F 1 "USB_C_Receptacle_USB2.0" H 6870 2548 50  0000 R CNN
-F 2 "Connector_USB:USB_C_Receptacle_XKB_U262-16XN-4BVC11" H 7450 2700 50  0001 C CNN
+F 2 "Connector_USB:USB_C_Receptacle_HRO_TYPE-C-31-M-12" H 7450 2700 50  0001 C CNN
 F 3 "https://www.usb.org/sites/default/files/documents/usb_type-c.zip" H 7450 2700 50  0001 C CNN
 	1    7300 2700
