File: Core/MIDI_USB.kicad_pcb (KiCad board)
At the start: 4 copper layers, 37.8 x 99.8 mm, 127 parts, among them J1 Conn_01x04, J10 AudioJack3_SwitchTR, J4 Conn_01x06, J5 USB_C_Receptacle_USB2.0, J6 Conn_02x08_Odd_Even, J7 AudioJack3_SwitchTR, J8 AudioJack3_SwitchTR, J9 AudioJack3_SwitchTR, Q1 ZXMP3A13, Q2 PMV88ENER, Q3 MMBT3904, Q5 ZXMP3A13, Q6 MMBT3904, SW1 SW_Push_DPDT, SW2 SW_SPST, SW3 SW_SPST, SW4 SW_SPST, U1 RP2040, U10 TLE9250V, U11 CAT250640VI, U12 APS1604M, U2 IS25LP032D, U4 TL072, U5 MIC5504-3.3YM5, U6 ES9023P, U7 PCM1808, U8 TL072, U9 MCP2517FD-xSL, Y1 20MHz, Y2 ECS-120-18-33-JGN-TR3

Commit message: Add optional solder bridge++
Parts:
- added NT1: NetTie_2, Jumper:SolderJumper-2_P1.3mm_Open_RoundedPad1.0x1.5mm, B.Cu at (158.0, 174.2)
Connections:
- J7 pad TN: unconnected-(J7-PadTN) -> Net-(J7-PadTN)
- J8 pad R: unconnected-(J8-PadR) -> Net-(J8-PadR)
Routing:
- net Net-(J7-PadTN): track 0.00 -> 8.26 mm
- net Net-(J8-PadR): track 0.00 -> 6.41 mm
Other:
- board text added: "TRS - L"
Changed lines of the file:
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@@
   (net 75 "unconnected-(J7-PadR)")
   (net 76 "unconnected-(J7-PadRN)")
-  (net 77 "unconnected-(J7-PadTN)")
-  (net 78 "unconnected-(J8-PadR)")
+  (net 77 "Net-(J7-PadTN)")
+  (net 78 "Net-(J8-PadR)")
   (net 79 "unconnected-(J8-PadRN)")
   (net 80 "unconnected-(J8-PadTN)")
@@
       (net 28 "Net-(J7-PadT)") (pintype "passive"))
     (pad "TN" thru_hole oval locked (at -2.5 5 180) (size 2.5 1.55) (drill oval 1.75 0.8) (layers "*.Cu" "*.Mask")
-      (net 77 "unconnected-(J7-PadTN)") (pintype "passive"))
+      (net 77 "Net-(J7-PadTN)") (pintype "passive"))
   )
   (footprint "Custom_FP:STX3100_Angled_3.5mm" locked (layer "F.Cu")
@@
     (pad "" np_thru_hole circle locked (at 5 0) (size 2 2) (drill 1.5) (layers "*.Cu" "*.Mask"))
     (pad "R" thru_hole oval locked (at 5 5) (size 2.5 1.55) (drill oval 1.75 0.8) (layers "*.Cu" "*.Mask")
-      (net 78 "unconnected-(J8-PadR)") (pintype "passive"))
+      (net 78 "Net-(J8-PadR)") (pintype "passive"))
     (pad "RN" thru_hole oval locked (at 2.5 5) (size 2.5 1.55) (drill oval 1.75 0.8) (layers "*.Cu" "*.Mask")
       (net 79 "unconnected-(J8-PadRN)") (pintype "passive"))
@@
     )
   )
+  (footprint "Jumper:SolderJumper-2_P1.3mm_Open_RoundedPad1.0x1.5mm" (layer "B.Cu")
+    (at 158 174.25 90)
+    (descr "SMD Solder Jumper, 1x1.5mm, rounded Pads, 0.3mm gap, open")
+    (tags "solder jumper open")
+    (property "Sheetfile" "Analog.kicad_sch")
+    (property "Sheetname" "Analog")
+    (property "exclude_from_bom" "")
+    (property "ki_description" "Net tie, 2 pins")
+    (property "ki_keywords" "net tie short")
+    (attr exclude_from_pos_files exclude_from_bom)
+    (fp_text reference "NT1" (at 0 1.8 90) (layer "B.SilkS") hide
+        (effects (font (size 1 1) (thickness 0.15)) (justify mirror))
+    )
+    (fp_text value "NetTie_2" (at 0 -1.9 90) (layer "B.Fab")
+        (effects (font (size 1 1) (thickness 0.15)) (justify mirror))
+    )
+    (fp_line (start -1.4 -0.3) (end -1.4 0.3)
+      (stroke (width 0.12) (type solid)) (layer "B.SilkS"))
+    (fp_line (start -0.7 1) (end 0.7 1)
+      (stroke (width 0.12) (type solid)) (layer "B.SilkS"))
+    (fp_line (start 0.7 -1) (end -0.7 -1)
+      (stroke (width 0.12) (type solid)) (layer "B.SilkS"))
+    (fp_line (start 1.4 0.3) (end 1.4 -0.3)
+      (stroke (width 0.12) (type solid)) (layer "B.SilkS"))
+    (fp_arc (start -1.4 -0.3) (mid -1.194975 -0.794975) (end -0.7 -1)
+      (stroke (width 0.12) (type solid)) (layer "B.SilkS"))
+    (fp_arc (start -0.7 1) (mid -1.194975 0.794975) (end -1.4 0.3)
+      (stroke (width 0.12) (type solid)) (layer "B.SilkS"))
+    (fp_arc (start 0.7 -1) (mid 1.194975 -0.794975) (end 1.4 -0.3)
+      (stroke (width 0.12) (type solid)) (layer "B.SilkS"))
+    (fp_arc (start 1.4 0.3) (mid 1.194975 0.794975) (end 0.7 1)
+      (stroke (width 0.12) (type solid)) (layer "B.SilkS"))
+    (fp_line (start -1.65 1.25) (end -1.65 -1.25)
+      (stroke (width 0.05) (type solid)) (layer "B.CrtYd"))
+    (fp_line (start -1.65 1.25) (end 1.65 1.25)
+      (stroke (width 0.05) (type solid)) (layer "B.CrtYd"))
+    (fp_line (start 1.65 -1.25) (end -1.65 -1.25)
+      (stroke (width 0.05) (type solid)) (layer "B.CrtYd"))
+    (fp_line (start 1.65 -1.25) (end 1.65 1.25)
+      (stroke (width 0.05) (type solid)) (layer "B.CrtYd"))
+    (pad "1" smd custom (at -0.65 0 90) (size 1 0.5) (layers "B.Cu" "B.Mask")
+      (net 77 "Net-(J7-PadTN)") (pinfunction "1") (pintype "passive") (zone_connect 2) (thermal_bridge_angle 45)
+      (options (clearance outline) (anchor rect))
+      (primitives
+        (gr_circle (center 0 -0.25) (end 0.5 -0.25) (width 0) (fill yes))
+        (gr_circle (center 0 0.25) (end 0.5 0.25) (width 0) (fill yes))
+        (gr_poly
+          (pts
+            (xy 0.5 -0.75)
+            (xy 0 -0.75)
+            (xy 0 0.75)
+            (xy 0.5 0.75)
+          )
+          (width 0) (fill yes))
+      ))
+    (pad "2" smd custom (at 0.65 0 90) (size 1 0.5) (layers "B.Cu" "B.Mask")
+      (net 78 "Net-(J8-PadR)") (pinfunction "2") (pintype "passive") (zone_connect 2) (thermal_bridge_angle 45)
+      (options (clearance outline) (anchor rect))
+      (primitives
+        (gr_circle (center 0 -0.25) (end 0.5 -0.25) (width 0) (fill yes))
+        (gr_circle (center 0 0.25) (end 0.5 0.25) (width 0) (fill yes))
+        (gr_poly
+          (pts
+            (xy 0 -0.75)
+            (xy -0.5 -0.75)
+            (xy -0.5 0.75)
+            (xy 0 0.75)
+          )
+          (width 0) (fill yes))
+      ))
+  )
   (footprint "Capacitor_SMD:C_0603_1608Metric" (layer "B.Cu")
     (at 162.25 123.375 45)
@@
     )
   )
+  (gr_rect (start 153.75 169) (end 159.75 180)
+    (stroke (width 0.12) (type default)) (fill none) (layer "B.SilkS"))
   (gr_line (start 143.25 110.25) (end 143.25 109)
     (stroke (width 0.12) (type solid)) (layer "F.SilkS"))
@@
     (effects (font (size 1 1) (thickness 0.15)) (justify mirror))
   )
+  (gr_text "TRS - L" (at 154.25 179.5 -90) (layer "B.SilkS")
+    (effects (font (size 1.6 1.6) (thickness 0.15)) (justify left bottom mirror))
+  )
   (gr_text "RESET" (at 134.1 124.925) (layer "F.SilkS")
     (effects (font (size 1.6 1.6) (thickness 0.15)) (justify left bottom))
@@
   (segment (start 152.927899 123.410742) (end 152.267156 122.75) (width 0.2) (layer "B.Cu") (net 71))
   (segment (start 151.15 122.75) (end 150.733363 122.333363) (width 0.2) (layer "B.Cu") (net 71))
+  (segment (start 163 178.75) (end 159 178.75) (width 0.25) (layer "B.Cu") (net 77))
+  (segment (start 158 177.75) (end 158 174.9) (width 0.25) (layer "B.Cu") (net 77))
+  (segment (start 159 178.75) (end 158 177.75) (width 0.25) (layer "B.Cu") (net 77))
+  (segment (start 158 172.5) (end 158.75 171.75) (width 0.25) (layer "B.Cu") (net 78))
+  (segment (start 158 173.6) (end 158 172.5) (width 0.25) (layer "B.Cu") (net 78))
+  (segment (start 158.75 171.75) (end 163 171.75) (width 0.25) (layer "B.Cu") (net 78))
   (segment (start 159.075 120.9625) (end 160.2375 120.9625) (width 0.25) (layer "F.Cu") (net 83))
   (segment (start 160.2375 120.9625) (end 162.025 119.175) (width 0.25) (layer "F.Cu") (net 83))
