File: Core/MIDI_USB.kicad_pcb (KiCad board)
At the start: 4 copper layers, 37.8 x 99.8 mm, 128 parts, among them J1 Conn_01x04, J10 AudioJack3_SwitchTR, J4 Conn_01x06, J5 USB_C_Receptacle_USB2.0, J6 Conn_02x08_Odd_Even, J7 AudioJack3_SwitchTR, J8 AudioJack3_SwitchTR, J9 AudioJack3_SwitchTR, Q1 ZXMP3A13, Q2 PMV88ENER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

Commit message: Change CAN tranceiver to MCP2562
Parts:
- U10: value TLE9250V -> MCP2562FD-ESN; footprint Package_SO:Infineon_PG-DSO-8-27_3.9x4.9mm_EP2.65x3mm -> Package_SO:SOIC-8_3.9x4.9mm_P1.27mm
- U13: value ~ -> TPS25820
Changed lines of the file:
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@@
         (effects (font (size 1 1) (thickness 0.15)))
     )
-    (fp_text value "~" (at 0 2.921) (layer "F.Fab")
+    (fp_text value "TPS25820" (at 0 2.921) (layer "F.Fab")
         (effects (font (size 1 1) (thickness 0.15)))
     )
@@
     )
   )
-  (footprint "Package_SO:Infineon_PG-DSO-8-27_3.9x4.9mm_EP2.65x3mm" (layer "B.Cu")
+  (footprint "Package_SO:SOIC-8_3.9x4.9mm_P1.27mm" (layer "B.Cu")
     (at 137.8 115.2 90)
-    (descr "Infineon  PG-DSO, 8 Pin (https://www.infineon.com/cms/en/product/packages/PG-DSO/PG-DSO-8-27), generated with kicad-footprint-generator ipc_gullwing_generator.py")
-    (tags "Infineon PG-DSO SO")
+    (descr "SOIC, 8 Pin (JEDEC MS-012AA, https://www.analog.com/media/en/package-pcb-resources/package/pkg_pdf/soic_narrow-r/r_8.pdf), generated with kicad-footprint-generator ipc_gullwing_generator.py")
+    (tags "SOIC SO")
     (property "Sheetfile" "MIDI_USB.kicad_sch")
     (property "Sheetname" "")
-    (property "ki_description" "CAN FD Transceiver with Silent Mode, up to 8 Mbps, DFN-8")
-    (property "ki_keywords" "CAN FD Transceiver")
-    (attr smd)
-    (fp_text reference "U10" (at 0 3.4 90) (layer "B.SilkS")
-        (effects (font (size 1 1) (thickness 0.15)) (justify mirror))
-    )
-    (fp_text value "TLE9250V" (at 0 -3.4 90) (layer "B.Fab")
-        (effects (font (size 1 1) (thickness 0.15)) (justify mirror))
-    )
-    (fp_text user "${REFERENCE}" (at 0 0 90) (layer "B.Fab")
+    (property "ki_description" "High-Speed CAN Transceiver, 1Mbps, 5V supply, Vio pin, -40C to +125C, SOIC-8")
+    (property "ki_keywords" "High-Speed CAN Transceiver")
+    (attr smd)
+    (fp_text reference "U10" (at 0 3.4 270) (layer "B.SilkS")
+        (effects (font (size 1 1) (thickness 0.15)) (justify mirror))
+    )
+    (fp_text value "MCP2562FD-ESN" (at 0 -3.4 270) (layer "B.Fab")
+        (effects (font (size 1 1) (thickness 0.15)) (justify mirror))
+    )
+    (fp_text user "${REFERENCE}" (at 0 0 270) (layer "B.Fab")
         (effects (font (size 0.98 0.98) (thickness 0.15)) (justify mirror))
     )
@@
     (fp_line (start 1.95 2.45) (end 1.95 -2.45)
       (stroke (width 0.1) (type solid)) (layer "B.Fab"))
-    (pad "" smd roundrect (at -0.66 -0.75 90) (size 1.07 1.21) (layers "B.Paste") (roundrect_rratio 0.233645))
-    (pad "" smd roundrect (at -0.66 0.75 90) (size 1.07 1.21) (layers "B.Paste") (roundrect_rratio 0.233645))
-    (pad "" smd roundrect (at 0.66 -0.75 90) (size 1.07 1.21) (layers "B.Paste") (roundrect_rratio 0.233645))
-    (pad "" smd roundrect (at 0.66 0.75 90) (size 1.07 1.21) (layers "B.Paste") (roundrect_rratio 0.233645))
-    (pad "1" smd roundrect (at -2.625 1.905 90) (size 1.65 0.6) (layers "B.Cu" "B.Paste" "B.Mask") (roundrect_rratio 0.25)
+    (pad "1" smd roundrect (at -2.475 1.905 90) (size 1.95 0.6) (layers "B.Cu" "B.Paste" "B.Mask") (roundrect_rratio 0.25)
       (net 109 "Net-(U10-TXD)") (pinfunction "TXD") (pintype "input"))
-    (pad "2" smd roundrect (at -2.625 0.635 90) (size 1.65 0.6) (layers "B.Cu" "B.Paste" "B.Mask") (roundrect_rratio 0.25)
+    (pad "2" smd roundrect (at -2.475 0.635 90) (size 1.95 0.6) (layers "B.Cu" "B.Paste" "B.Mask") (roundrect_rratio 0.25)
       (net 1 "GND") (pinfunction "VSS") (pintype "power_in"))
-    (pad "3" smd roundrect (at -2.625 -0.635 90) (size 1.65 0.6) (layers "B.Cu" "B.Paste" "B.Mask") (roundrect_rratio 0.25)
+    (pad "3" smd roundrect (at -2.475 -0.635 90) (size 1.95 0.6) (layers "B.Cu" "B.Paste" "B.Mask") (roundrect_rratio 0.25)
       (net 3 "+5V") (pinfunction "VDD") (pintype "power_in"))
-    (pad "4" smd roundrect (at -2.625 -1.905 90) (size 1.65 0.6) (layers "B.Cu" "B.Paste" "B.Mask") (roundrect_rratio 0.25)
+    (pad "4" smd roundrect (at -2.475 -1.905 90) (size 1.95 0.6) (layers "B.Cu" "B.Paste" "B.Mask") (roundrect_rratio 0.25)
       (net 110 "Net-(U10-RXD)") (pinfunction "RXD") (pintype "output"))
-    (pad "5" smd roundrect (at 2.625 -1.905 90) (size 1.65 0.6) (layers "B.Cu" "B.Paste" "B.Mask") (roundrect_rratio 0.25)
-      (net 8 "+3V3") (pinfunction "VIO") (pintype "power_in"))
-    (pad "6" smd roundrect (at 2.625 -0.635 90) (size 1.65 0.6) (layers "B.Cu" "B.Paste" "B.Mask") (roundrect_rratio 0.25)
+    (pad "5" smd roundrect (at 2.475 -1.905 90) (size 1.95 0.6) (layers "B.Cu" "B.Paste" "B.Mask") (roundrect_rratio 0.25)
+      (net 8 "+3V3") (pinfunction "Vio") (pintype "power_in"))
+    (pad "6" smd roundrect (at 2.475 -0.635 90) (size 1.95 0.6) (layers "B.Cu" "B.Paste" "B.Mask") (roundrect_rratio 0.25)
       (net 43 "M2IDI-") (pinfunction "CANL") (pintype "bidirectional"))
-    (pad "7" smd roundrect (at 2.625 0.635 90) (size 1.65 0.6) (layers "B.Cu" "B.Paste" "B.Mask") (roundrect_rratio 0.25)
+    (pad "7" smd roundrect (at 2.475 0.635 90) (size 1.95 0.6) (layers "B.Cu" "B.Paste" "B.Mask") (roundrect_rratio 0.25)
       (net 44 "M2IDI+") (pinfunction "CANH") (pintype "bidirectional"))
-    (pad "8" smd roundrect (at 2.625 1.905 90) (size 1.65 0.6) (layers "B.Cu" "B.Paste" "B.Mask") (roundrect_rratio 0.25)
-      (net 1 "GND") (pinfunction "S") (pintype "input"))
-    (pad "9" smd rect (at 0 0 90) (size 2.65 3) (layers "B.Cu" "B.Mask")
-      (net 1 "GND") (pinfunction "VSS") (pintype "passive"))
-    (model "${KICAD6_3DMODEL_DIR}/Package_SO.3dshapes/Infineon_PG-DSO-8-27_3.9x4.9mm_EP2.65x3mm.wrl"
+    (pad "8" smd roundrect (at 2.475 1.905 90) (size 1.95 0.6) (layers "B.Cu" "B.Paste" "B.Mask") (roundrect_rratio 0.25)
+      (net 1 "GND") (pinfunction "STBY") (pintype "input"))
+    (model "${KICAD6_3DMODEL_DIR}/Package_SO.3dshapes/SOIC-8_3.9x4.9mm_P1.27mm.wrl"
       (offset (xyz 0 0 0))
       (scale (xyz 1 1 1))
@@
     (property "ki_description" "Two pin crystal")
     (property "ki_keywords" "quartz ceramic resonator oscillator")
-    (attr through_hole)
+    (attr smd)
     (fp_text reference "Y1" (at -3.224 0.33) (layer "B.SilkS")
         (effects (font (size 1 1) (thickness 0.15)) (justify mirror))
